File: rev-0.2/kicad/design.sch (KiCad schematic (older format))
At the start: 21 parts, among them P1 AUX-4_INTERFACE, P2 I2C_INTERFACE, P3 PROGRAM_JUMPERS, U1 RN-171, U2 TXB0106PWR, U3 LM358DMR2G, U4 TC1262-3.3VDB

Commit message: Changing R6,R8 to 4.7KOhm and R7,R9 to 9.1KOhm. Removing unused libraries from Eeschema. Updating and fixing some errors in BOM.
Parts:
- removed R6, R8: CR0805-FX-4702ELF, symbol CR0805-FX-4702ELF
- removed R7, R9: CR0805-FX-9102ELF, symbol CR0805-FX-9102ELF
- added R6, R8: CR0805-FX-4701ELF, symbol CR0805-FX-4701ELF
- added R7, R9: CR0805-FX-9101ELF, symbol CR0805-FX-9101ELF
Changed lines of the file:
@@
-EESchema Schematic File Version 2  date Wed 19 Jun 2013 11:22:25 AM CDT
+EESchema Schematic File Version 2  date Tue 03 Sep 2013 03:17:11 PM CDT
 LIBS:power
 LIBS:device
@@
 LIBS:_roving_networks_
 LIBS:_microchip_
-LIBS:_vishay_
-LIBS:_panasonic_
 LIBS:_texas_instruments_
 LIBS:_headers_
@@
 Sheet 1 1
 Title "RAMPS WiFi Adapter"
-Date "18 jun 2013"
+Date "3 sep 2013"
 Rev ".2"
 Comp "ODDepot.com, Finucane Design LLC"
@@
 	6600 4800 6700 4800
 $Comp
-L CR0805-FX-4702ELF R6
-U 1 1 51B5DF5A
-P 2950 1150
-F 0 "R6" H 2950 1250 50  0000 C CNN
-F 1 "CR0805-FX-4702ELF" H 2950 1050 50  0000 C CNN
-F 4 "47_KOHM" H 2950 950 50  0000 C CNN "Description"
-	1    2950 1150
-	1    0    0    -1
-$EndComp
-$Comp
-L CR0805-FX-9102ELF R7
-U 1 1 51B5DF73
-P 3850 1150
-F 0 "R7" H 3850 1250 50  0000 C CNN
-F 1 "CR0805-FX-9102ELF" H 3850 1050 50  0000 C CNN
-F 4 "91_KOHM" H 3850 950 50  0000 C CNN "Description"
-	1    3850 1150
-	1    0    0    -1
-$EndComp
-$Comp
 L GND #PWR4
 U 1 1 51B5DF8C
@@
 	1    4200 1150
 	0    -1   -1   0
-$EndComp
-$Comp
-L CR0805-FX-4702ELF R8
-U 1 1 51B5E50E
-P 2950 2150
-F 0 "R8" H 2950 2250 50  0000 C CNN
-F 1 "CR0805-FX-4702ELF" H 2950 2050 50  0000 C CNN
-F 4 "47_KOHM" H 2950 1950 50  0000 C CNN "Description"
-	1    2950 2150
-	1    0    0    -1
-$EndComp
-$Comp
-L CR0805-FX-9102ELF R9
-U 1 1 51B5E515
-P 3850 2150
-F 0 "R9" H 3850 2250 50  0000 C CNN
-F 1 "CR0805-FX-9102ELF" H 3850 2050 50  0000 C CNN
-F 4 "91_KOHM" H 3850 1950 50  0000 C CNN "Description"
-	1    3850 2150
-	1    0    0    -1
 $EndComp
 $Comp
@@
 Text Label 4900 4550 0    50   ~ 0
 DFLT
+$Comp
+L CR0805-FX-4701ELF R6
+U 1 1 522643D6
+P 2950 1150
+F 0 "R6" H 2950 1250 50  0000 C CNN
+F 1 "CR0805-FX-4701ELF" H 2950 1050 50  0000 C CNN
+F 4 "4.7_KOHM" H 2950 950 50  0000 C CNN "Description"
+	1    2950 1150
+	1    0    0    -1
+$EndComp
+$Comp
+L CR0805-FX-4701ELF R8
+U 1 1 522643EF
+P 2950 2150
+F 0 "R8" H 2950 2250 50  0000 C CNN
+F 1 "CR0805-FX-4701ELF" H 2950 2050 50  0000 C CNN
+F 4 "4.7_KOHM" H 2950 1950 50  0000 C CNN "Description"
+	1    2950 2150
+	1    0    0    -1
+$EndComp
+$Comp
+L CR0805-FX-9101ELF R7
+U 1 1 52264414
+P 3850 1150
+F 0 "R7" H 3850 1250 50  0000 C CNN
+F 1 "CR0805-FX-9101ELF" H 3850 1050 50  0000 C CNN
+F 4 "9.1_KOHM" H 3850 950 50  0000 C CNN "Description"
+	1    3850 1150
+	1    0    0    -1
+$EndComp
+$Comp
+L CR0805-FX-9101ELF R9
+U 1 1 5226442D
+P 3850 2150
+F 0 "R9" H 3850 2250 50  0000 C CNN
+F 1 "CR0805-FX-9101ELF" H 3850 2050 50  0000 C CNN
+F 4 "9.1_KOHM" H 3850 1950 50  0000 C CNN "Description"
+	1    3850 2150
+	1    0    0    -1
+$EndComp
 $EndSCHEMATC
